Commit message: added inertia to table model in UR5 single arm xacro file

File: ur5_single_arm_tufts/urdf/ur5_single_arm.xacro (robot description, xacro)
@@ -23,4 +23,12 @@
       </geometry>
     </visual>
+    <inertial>
+      <origin xyz="0.23 0 0.755" rpy="0 0 0" />
+      <mass value="1"/>
+      <inertia
+        ixx="0.07" ixy="0.0" ixz="0.0"
+        iyy="0.40" iyz="0.0"
+        izz="0.33"/>
+    </inertial>
     <collision>
       <geometry>

Commit message: Updated urdf model with good physics

File: ur5_single_arm_tufts/urdf/ur5_single_arm.xacro (robot description, xacro)
@@ -23,5 +23,5 @@
       </geometry>
     </visual>
-    <inertial>
+     <inertial>
       <origin xyz="0.23 0 0.755" rpy="0 0 0" />
       <mass value="1"/>
