Commit message: robot des. Version 2

File: ur5_single_arm_tufts/urdf/ur5_single_arm.urdf (robot description, URDF)
Before this commit: robot ur5, 21 links, 20 joints
Links:
- removed link table
- added link robot_pilar, mass 1; collision cylinder length=0.9 radius=0.1; visual cylinder length=0.9 radius=0.1
- added link table_base, mass 12.6503207764878; collision mesh filename=package://ur5_single_arm_tufts/meshes/objects/table_base.STL; visual mesh filename=package://ur5_single_arm_tufts/meshes/objects/table_base.STL
- added link table_top, mass 27.72; collision box size=0.005 0.015 0.8; collision box size=1.05 0.015 0.005
- added link tabletop_corner
- added link tabletop_ontop
Joints:
- removed joint table_to_robot
- removed joint world_to_table
- added joint j1: type fixed, parent table_base, child table_top, origin xyz=0.0185115091791201 -0.175991980646074 0.397575968372377 rpy=1.5707963267949 0 0, axis 0 0 0
- added joint pilar_to_world: type fixed, parent world, child robot_pilar, origin xyz=0 0 0.45 rpy=0 0 0
- added joint robot_to_pilar: type fixed, parent robot_pilar, child base_link, origin xyz=0 0 0.45 rpy=0 0 0
- added joint set_tabletop_relto_corner: type fixed, parent tabletop_ontop, child tabletop_corner, origin xyz=0.42 0.3 0 rpy=0 0 -0.76
- added joint table_tabletop_totop: type fixed, parent table_top, child tabletop_ontop, origin xyz=0.0 0.033 0 rpy=-1.57079632679 0 0, axis 0 0 0
- added joint table_to_world: type fixed, parent world, child table_base, origin xyz=0.9 0.08 0.3 rpy=0 0 -1.555
- joint shoulder_lift_joint: limit lower=-3.14159265359 upper=3.14159265359 effort=150.0 velocity=3.15 -> lower=-6.28318530718 upper=6.28318530718 effort=150.0 velocity=3.15
- joint shoulder_pan_joint: limit lower=-3.14159265359 upper=3.14159265359 effort=150.0 velocity=3.15 -> lower=-6.28318530718 upper=6.28318530718 effort=150.0 velocity=3.15
- joint wrist_1_joint: limit lower=-3.14159265359 upper=3.14159265359 effort=28.0 velocity=3.2 -> lower=-6.28318530718 upper=6.28318530718 effort=28.0 velocity=3.2
- joint wrist_2_joint: limit lower=-3.14159265359 upper=3.14159265359 effort=28.0 velocity=3.2 -> lower=-6.28318530718 upper=6.28318530718 effort=28.0 velocity=3.2
- joint wrist_3_joint: limit lower=-3.14159265359 upper=3.14159265359 effort=28.0 velocity=3.2 -> lower=-6.28318530718 upper=6.28318530718 effort=28.0 velocity=3.2

Commit message: Added Grasp Fix

File: ur5_single_arm_tufts/urdf/ur5_single_arm.urdf (robot description, URDF)
Before this commit: robot ur5, 25 links, 24 joints
Links:
- removed link table_base
- removed link table_top
- removed link tabletop_corner
- removed link tabletop_ontop
- link robot_pilar: geometry collision cylinder length=0.9 radius=0.07; visual cylinder length=0.9 radius=0.07
Joints:
- removed joint j1
- removed joint set_tabletop_relto_corner
- removed joint table_tabletop_totop
- removed joint table_to_world

File: ur5_single_arm_tufts/urdf/ur5_single_arm.urdf.xacro (robot description, xacro)
@@ -13,4 +13,9 @@
     <origin xyz="0 0 0" rpy="0 0 0"/>
   </xacro:robotiq_85_gripper>
+    <!-- kinect -->
+<!--   <xacro:include filename="$(find ur5_single_arm_tufts)/urdf/sensors/kinect/kinect.urdf.xacro" />
+  <xacro:kinect name="camera" parent="world" >
+    <origin xyz="0.4 0.0 1.2" rpy="0.0 ${pi/2} 0.0" />
+  </xacro:kinect> -->
   <!-- kinect, ir, rgb sensor-->
 <!--   <xacro:include filename="$(find ur5_single_arm_tufts)/urdf/sensors/kinect2/common.xacro" />
@@ -19,14 +24,9 @@
     <origin xyz="0.4 0.0 1.2" rpy="0.0 ${pi/2} 0.0" />
   </xacro:kinect2_v0> -->
-  <!-- kinect -->
-  <xacro:include filename="$(find ur5_single_arm_tufts)/urdf/sensors/kinect/kinect.urdf.xacro" />
-  <xacro:kinect name="camera" parent="world" >
-    <origin xyz="0.4 0.0 1.2" rpy="0.0 ${pi/2} 0.0" />
-  </xacro:kinect>
   <!-- Pilar property -->
   <xacro:property name="pilar_height" value="0.9"/>
   <xacro:property name="pilar_radius" value="0.07"/>
   <link name="world"/>
-  <link name="table">
+<!--   <link name="table">
     <inertial>
       <origin xyz="0.23 0 0.755" rpy="0 0 0" />
@@ -54,7 +54,6 @@
       <parent link="world"/>
       <child link="table"/>
-      <!-- <origin xyz="0.85 0 0.7" rpy="0 0 0"/> -->
-      <origin xyz="0.85 0 0.72" rpy="0 0 0"/>
-  </joint>
+      <origin xyz="0.85 0 0.70" rpy="0 0 0"/>
+  </joint> -->
   <link name="robot_pilar">
     <visual>
@@ -89,3 +88,5 @@
     <origin xyz="0 0 ${pilar_height/2}" rpy="0 0 0"/>
   </joint>
+  <xacro:include filename="$(find ur5_single_arm_tufts)/urdf/gzplugin_grasp_fix.urdf.xacro"/>
+  <xacro:gzplugin_grasp_fix/>
 </robot>
