Commit message: Added pick and place demo

File: ur5_single_arm_tufts/urdf/gzplugin_grasp_fix.urdf.xacro (robot description, xacro)
@@ -16,10 +16,11 @@
             <arm>
                 <arm_name>UR5Arm</arm_name>
-<!--                 <palm_link> robotiq_85_left_inner_knuckle_link </palm_link>
-		        <gripper_link> robotiq_85_left_finger_tip_link </gripper_link>
-		        <palm_link> robotiq_85_right_knuckle_link </palm_link>
-		        <gripper_link> robotiq_85_right_finger_tip_link </gripper_link>
- -->
-                <palm_link>wrist_3_link</palm_link>
+                <!-- 0.01977<0.0198<0.01999 -->
+                <palm_link> gripper_finger1_inner_knuckle_link </palm_link>
+		        <gripper_link> gripper_finger1_finger_tip_link </gripper_link>
+		        <palm_link> gripper_finger2_inner_knuckle_link </palm_link>
+		        <gripper_link> gripper_finger2_finger_tip_link </gripper_link>
+		        <!-- 0.01976<0.01977<0.01978 -->
+<!--                 <palm_link>wrist_3_link</palm_link>
                 <gripper_link>gripper_finger1_inner_knuckle_link</gripper_link>
                 <gripper_link>gripper_finger1_finger_tip_link</gripper_link>
@@ -28,10 +29,11 @@
                 <gripper_link>gripper_finger2_finger_tip_link</gripper_link>
                 <gripper_link>gripper_finger2_knuckle_link</gripper_link>
+ -->
             </arm>
 			<forces_angle_tolerance>100</forces_angle_tolerance>
-			<update_rate>4</update_rate>
-			<grip_count_threshold>4</grip_count_threshold>
-			<max_grip_count>8</max_grip_count>
-			<release_tolerance>0.005</release_tolerance>
+			<update_rate>20</update_rate>
+			<grip_count_threshold>1</grip_count_threshold>
+			<max_grip_count>3</max_grip_count>
+			<release_tolerance>0.0198</release_tolerance> <!-- 0.01977<0.0198<0.01999 -->
 			<disable_collisions_on_attach>false</disable_collisions_on_attach>
 			<contact_topic>__default_topic__</contact_topic>

File: ur5_single_arm_tufts/urdf/ur5_single_arm.urdf.xacro (robot description, xacro)
@@ -14,8 +14,8 @@
   </xacro:robotiq_85_gripper>
     <!-- kinect -->
-<!--   <xacro:include filename="$(find ur5_single_arm_tufts)/urdf/sensors/kinect/kinect.urdf.xacro" />
+  <xacro:include filename="$(find ur5_single_arm_tufts)/urdf/sensors/kinect/kinect.urdf.xacro" />
   <xacro:kinect name="camera" parent="world" >
-    <origin xyz="0.4 0.0 1.2" rpy="0.0 ${pi/2} 0.0" />
-  </xacro:kinect> -->
+    <origin xyz="0.6 0.0 1.8" rpy="0.0 ${pi/2} 0.0" />
+  </xacro:kinect>
   <!-- kinect, ir, rgb sensor-->
 <!--   <xacro:include filename="$(find ur5_single_arm_tufts)/urdf/sensors/kinect2/common.xacro" />
