Commit message: updated arm positions on ur5frame

File: ur5_dual_arm_tufts/urdf/ur5_dual_arm.xacro (robot description, xacro)
@@ -42,10 +42,10 @@
     <parent link="ur5_frame" />
     <child link = "base_link" />
-    <origin xyz="0.607 0.635 1.27" rpy="${0*pi/180} ${135*pi/180}  ${0*pi/180}" />
+    <origin xyz="0.645 0.635 1.275" rpy="${0*pi/180} ${135*pi/180}  ${0*pi/180}" />
   </joint>
   <joint name="world_joint_2" type="fixed">
     <parent link="ur5_frame" />
     <child link = "2_base_link" />
-    <origin xyz="0.28 0.69 1.27" rpy="${0*pi/180} ${225*pi/180}  ${0*pi/180}" />
+    <origin xyz="0.265 0.635 1.275" rpy="${0*pi/180} ${225*pi/180}  ${0*pi/180}" />
   </joint>
   <!-- robotiq 85 1 -->

Commit message: updated collision inertia properties for UR5 frame

File: ur5_dual_arm_tufts/urdf/ur5_dual_arm.xacro (robot description, xacro)
@@ -27,4 +27,18 @@
   <link name="world"/>
   <link name="ur5_frame">
+    <inertial>
+      <origin rpy  ="0.0 0 0" xyz="0 0 0"/>
+      <mass value="27.2155"/>
+      <inertia
+        ixx="5.01" ixy="0.0" ixz="0.0"
+        iyy="5.07" iyz="0.0"
+        izz="3.20"/>
+    </inertial>
+    <collision>
+      <origin rpy="0.0 0 0" xyz="0 0 0"/>
+      <geometry>
+        <mesh filename="package://ur5_dual_arm_tufts/meshes/UR5Frame.dae"/>
+      </geometry>
+    </collision>
     <visual>
       <origin rpy="0.0 0 0" xyz="0 0 0"/>

Commit message: updated dual arm parameters

File: ur5_dual_arm_tufts/urdf/ur5_dual_arm.xacro (robot description, xacro)
@@ -27,5 +27,5 @@
   <link name="world"/>
   <link name="ur5_frame">
-    <inertial>
+<!--     <inertial>
       <origin rpy  ="0.0 0 0" xyz="0 0 0"/>
       <mass value="27.2155"/>
@@ -34,11 +34,11 @@
         iyy="5.07" iyz="0.0"
         izz="3.20"/>
-    </inertial>
-    <collision>
+    </inertial> -->
+<!--     <collision>
       <origin rpy="0.0 0 0" xyz="0 0 0"/>
       <geometry>
         <mesh filename="package://ur5_dual_arm_tufts/meshes/UR5Frame.dae"/>
       </geometry>
-    </collision>
+    </collision> -->
     <visual>
       <origin rpy="0.0 0 0" xyz="0 0 0"/>

Commit message: updated yaml files

File: ur5_dual_arm_tufts/urdf/ur5_dual_arm.xacro (robot description, xacro)
@@ -27,5 +27,5 @@
   <link name="world"/>
   <link name="ur5_frame">
-<!--     <inertial>
+    <inertial>
       <origin rpy  ="0.0 0 0" xyz="0 0 0"/>
       <mass value="27.2155"/>
@@ -34,5 +34,5 @@
         iyy="5.07" iyz="0.0"
         izz="3.20"/>
-    </inertial> -->
+    </inertial>
 <!--     <collision>
       <origin rpy="0.0 0 0" xyz="0 0 0"/>
