Commit message: dual arm successful

File: ur5_dual_arm_tufts/urdf/ur5_dual_arm.xacro (robot description, xacro)
@@ -8,5 +8,5 @@
   <xacro:include filename="$(find robotiq_85_description)/urdf/robotiq_85_gripper.urdf.xacro" />
   <!-- arm 1 -->
-  <xacro:ur5_robot prefix="" joint_limited="true"
+  <xacro:ur5_robot prefix="right_" joint_limited="true"
     shoulder_pan_lower_limit="${-pi}" shoulder_pan_upper_limit="${pi}"
     shoulder_lift_lower_limit="${-pi}" shoulder_lift_upper_limit="${pi}"
@@ -17,5 +17,5 @@
   />
   <!-- arm 2 -->
-  <xacro:ur5_robot prefix="2_" joint_limited="true"
+  <xacro:ur5_robot prefix="left_" joint_limited="true"
     shoulder_pan_lower_limit="${-pi}" shoulder_pan_upper_limit="${pi}"
     shoulder_lift_lower_limit="${-pi}" shoulder_lift_upper_limit="${pi}"
@@ -53,22 +53,22 @@
     <origin xyz="0.0 0.0 0.0" rpy="0.0 0.0 0.0" />
   </joint>
-<!-- right arm -->
+<!-- left arm -->
   <joint name="world_joint_1" type="fixed">
     <parent link="ur5_frame" />
-    <child link = "base_link" />
+    <child link = "left_base_link" />
     <origin xyz="0.645 0.635 1.275" rpy="${0*pi/180} ${135*pi/180}  ${0*pi/180}" />
   </joint>
-<!-- left arm -->
+<!-- right arm -->
   <joint name="world_joint_2" type="fixed">
     <parent link="ur5_frame" />
-    <child link = "2_base_link" />
+    <child link = "right_base_link" />
     <origin xyz="0.265 0.635 1.275" rpy="${0*pi/180} ${225*pi/180}  ${0*pi/180}" />
   </joint>
-  <!-- robotiq 85 1 -->
-  <xacro:robotiq_85_gripper prefix="" parent="ee_link" >
+  <!-- robotiq 85 1 (left) -->
+  <xacro:robotiq_85_gripper prefix="left_" parent="left_ee_link" >
     <origin xyz="0 0 0" rpy="0 0 0"/>
   </xacro:robotiq_85_gripper>
-  <!-- robotiq 85 2 -->
-  <xacro:robotiq_85_gripper prefix="2_" parent="2_ee_link" >
+  <!-- robotiq 85 2 (right) -->
+  <xacro:robotiq_85_gripper prefix="right_" parent="right_ee_link" >
     <origin xyz="0 0 0" rpy="0 0 0"/>
   </xacro:robotiq_85_gripper>

File: ur5_dual_arm_tufts/urdf/ur5_dual_dre.urdf (robot description, URDF)
Before this commit: robot ur5, 40 links, 39 joints
Links:
- removed link 2_base
- removed link 2_base_link
- removed link 2_ee_link
- removed link 2_forearm_link
- removed link 2_gripper_base_link
- removed link 2_gripper_finger1_finger_link
- removed link 2_gripper_finger1_finger_tip_link
- removed link 2_gripper_finger1_inner_knuckle_link
- removed link 2_gripper_finger1_knuckle_link
- removed link 2_gripper_finger2_finger_link
- removed link 2_gripper_finger2_finger_tip_link
- removed link 2_gripper_finger2_inner_knuckle_link
- removed link 2_gripper_finger2_knuckle_link
- removed link 2_shoulder_link
- removed link 2_tool0
- removed link 2_upper_arm_link
- removed link 2_wrist_1_link
- removed link 2_wrist_2_link
- removed link 2_wrist_3_link
- removed link base
- removed link base_link
- removed link ee_link
- removed link forearm_link
- removed link gripper_base_link
- removed link gripper_finger1_finger_link
- removed link gripper_finger1_finger_tip_link
- removed link gripper_finger1_inner_knuckle_link
- removed link gripper_finger1_knuckle_link
- removed link gripper_finger2_finger_link
- removed link gripper_finger2_finger_tip_link
- removed link gripper_finger2_inner_knuckle_link
- removed link gripper_finger2_knuckle_link
- removed link shoulder_link
- removed link tool0
- removed link upper_arm_link
- removed link wrist_1_link
- removed link wrist_2_link
- removed link wrist_3_link
- added link left_base
- added link left_base_link, mass 4.0; collision mesh filename=package://ur_description/meshes/ur5/collision/base.stl; visual mesh filename=package://ur_description/meshes/ur5/visual/base.dae
- added link left_ee_link, mass 0.1; collision box size=0.01 0.01 0.01
- added link left_forearm_link, mass 2.275; collision mesh filename=package://ur_description/meshes/ur5/collision/forearm.stl; visual mesh filename=package://ur_description/meshes/ur5/visual/forearm.dae
- added link left_gripper_base_link, mass 0.636951; collision mesh filename=package://robotiq_85_description/meshes/collision/robotiq_8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; visual mesh filename=package://robotiq_85_description/meshes/visual/robotiq_85_b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
- added link left_gripper_finger1_finger_link, mass 0.027309; collision mesh filename=package://robotiq_85_description/meshes/collision/robotiq_8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; visual mesh filename=package://robotiq_85_description/meshes/visual/robotiq_85_f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
- added link left_gripper_finger1_finger_tip_link, mass 0.019555; collision mesh filename=package://robotiq_85_description/meshes/collision/robotiq_8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; visual mesh filename=package://robotiq_85_description/meshes/visual/robotiq_85_f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
- added link left_gripper_finger1_inner_knuckle_link, mass 0.029951; collision mesh filename=package://robotiq_85_description/meshes/collision/robotiq_8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; visual mesh filename=package://robotiq_85_description/meshes/visual/robotiq_85_i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
- added link left_gripper_finger1_knuckle_link, mass 0.018491; collision mesh filename=package://robotiq_85_description/meshes/collision/robotiq_8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; visual mesh filename=package://robotiq_85_description/meshes/visual/robotiq_85_k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
- added link left_gripper_finger2_finger_link, mass 0.027309; collision mesh filename=package://robotiq_85_description/meshes/collision/robotiq_8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; visual mesh filename=package://robotiq_85_description/meshes/visual/robotiq_85_f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
- added link left_gripper_finger2_finger_tip_link, mass 0.019555; collision mesh filename=package://robotiq_85_description/meshes/collision/robotiq_8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; visual mesh filename=package://robotiq_85_description/meshes/visual/robotiq_85_f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
- added link left_gripper_finger2_inner_knuckle_link, mass 0.029951; collision mesh filename=package://robotiq_85_description/meshes/collision/robotiq_8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; visual mesh filename=package://robotiq_85_description/meshes/visual/robotiq_85_i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
- added link left_gripper_finger2_knuckle_link, mass 0.018491; collision mesh filename=package://robotiq_85_description/meshes/collision/robotiq_8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; visual mesh filename=package://robotiq_85_description/meshes/visual/robotiq_85_k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
- added link left_shoulder_link, mass 3.7; collision mesh filename=package://ur_description/meshes/ur5/collision/shoulder.stl; visual mesh filename=package://ur_description/meshes/ur5/visual/shoulder.dae
- added link left_tool0
- added link left_upper_arm_link, mass 8.393; collision mesh filename=package://ur_description/meshes/ur5/collision/upperarm.stl; visual mesh filename=package://ur_description/meshes/ur5/visual/upperarm.dae
- added link left_wrist_1_link, mass 1.219; collision mesh filename=package://ur_description/meshes/ur5/collision/wrist1.stl; visual mesh filename=package://ur_description/meshes/ur5/visual/wrist1.dae
- added link left_wrist_2_link, mass 1.219; collision mesh filename=package://ur_description/meshes/ur5/collision/wrist2.stl; visual mesh filename=package://ur_description/meshes/ur5/visual/wrist2.dae
- added link left_wrist_3_link, mass 0.1879; collision mesh filename=package://ur_description/meshes/ur5/collision/wrist3.stl; visual mesh filename=package://ur_description/meshes/ur5/visual/wrist3.dae
- added link right_base
- added link right_base_link, mass 4.0; collision mesh filename=package://ur_description/meshes/ur5/collision/base.stl; visual mesh filename=package://ur_description/meshes/ur5/visual/base.dae
- added link right_ee_link, mass 0.1; collision box size=0.01 0.01 0.01
- added link right_forearm_link, mass 2.275; collision mesh filename=package://ur_description/meshes/ur5/collision/forearm.stl; visual mesh filename=package://ur_description/meshes/ur5/visual/forearm.dae
- added link right_gripper_base_link, mass 0.636951; collision mesh filename=package://robotiq_85_description/meshes/collision/robotiq_8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; visual mesh filename=package://robotiq_85_description/meshes/visual/robotiq_85_b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
- added link right_gripper_finger1_finger_link, mass 0.027309; collision mesh filename=package://robotiq_85_description/meshes/collision/robotiq_8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; visual mesh filename=package://robotiq_85_description/meshes/visual/robotiq_85_f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
- added link right_gripper_finger1_finger_tip_link, mass 0.019555; collision mesh filename=package://robotiq_85_description/meshes/collision/robotiq_8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; visual mesh filename=package://robotiq_85_description/meshes/visual/robotiq_85_f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
- added link right_gripper_finger1_inner_knuckle_link, mass 0.029951; collision mesh filename=package://robotiq_85_description/meshes/collision/robotiq_8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; visual mesh filename=package://robotiq_85_description/meshes/visual/robotiq_85_i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
- added link right_gripper_finger1_knuckle_link, mass 0.018491; collision mesh filename=package://robotiq_85_description/meshes/collision/robotiq_8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; visual mesh filename=package://robotiq_85_description/meshes/visual/robotiq_85_k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
- added link right_gripper_finger2_finger_link, mass 0.027309; collision mesh filename=package://robotiq_85_description/meshes/collision/robotiq_8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; visual mesh filename=package://robotiq_85_description/meshes/visual/robotiq_85_f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
- added link right_gripper_finger2_finger_tip_link, mass 0.019555; collision mesh filename=package://robotiq_85_description/meshes/collision/robotiq_8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; visual mesh filename=package://robotiq_85_description/meshes/visual/robotiq_85_f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
- added link right_gripper_finger2_inner_knuckle_link, mass 0.029951; collision mesh filename=package://robotiq_85_description/meshes/collision/robotiq_8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; visual mesh filename=package://robotiq_85_description/meshes/visual/robotiq_85_i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
- added link right_gripper_finger2_knuckle_link, mass 0.018491; collision mesh filename=package://robotiq_85_description/meshes/collision/robotiq_8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; visual mesh filename=package://robotiq_85_description/meshes/visual/robotiq_85_k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
- added link right_shoulder_link, mass 3.7; collision mesh filename=package://ur_description/meshes/ur5/collision/shoulder.stl; visual mesh filename=package://ur_description/meshes/ur5/visual/shoulder.dae
- added link right_tool0
- added link right_upper_arm_link, mass 8.393; collision mesh filename=package://ur_description/meshes/ur5/collision/upperarm.stl; visual mesh filename=package://ur_description/meshes/ur5/visual/upperarm.dae
- added link right_wrist_1_link, mass 1.219; collision mesh filename=package://ur_description/meshes/ur5/collision/wrist1.stl; visual mesh filename=package://ur_description/meshes/ur5/visual/wrist1.dae
- added link right_wrist_2_link, mass 1.219; collision mesh filename=package://ur_description/meshes/ur5/collision/wrist2.stl; visual mesh filename=package://ur_description/meshes/ur5/visual/wrist2.dae
- added link right_wrist_3_link, mass 0.1879; collision mesh filename=package://ur_description/meshes/ur5/collision/wrist3.stl; visual mesh filename=package://ur_description/meshes/ur5/visual/wrist3.dae
- link ur5_frame: mass None -> 27.2155
Joints:
- removed joint 2_base_link-base_fixed_joint
- removed joint 2_ee_fixed_joint
- removed joint 2_elbow_joint
- removed joint 2_gripper_base_joint
- removed joint 2_gripper_finger1_finger_joint
- removed joint 2_gripper_finger1_finger_tip_joint
- removed joint 2_gripper_finger1_inner_knuckle_joint
- removed joint 2_gripper_finger1_joint
- removed joint 2_gripper_finger2_finger_joint
- removed joint 2_gripper_finger2_finger_tip_joint
- removed joint 2_gripper_finger2_inner_knuckle_joint
- removed joint 2_gripper_finger2_joint
- removed joint 2_shoulder_lift_joint
- removed joint 2_shoulder_pan_joint
- removed joint 2_wrist_1_joint
- removed joint 2_wrist_2_joint
- removed joint 2_wrist_3_joint
- removed joint 2_wrist_3_link-tool0_fixed_joint
- removed joint base_link-base_fixed_joint
- removed joint ee_fixed_joint
- removed joint elbow_joint
- removed joint gripper_base_joint
- removed joint gripper_finger1_finger_joint
- removed joint gripper_finger1_finger_tip_joint
- removed joint gripper_finger1_inner_knuckle_joint
- removed joint gripper_finger1_joint
- removed joint gripper_finger2_finger_joint
- removed joint gripper_finger2_finger_tip_joint
- removed joint gripper_finger2_inner_knuckle_joint
- removed joint gripper_finger2_joint
- removed joint shoulder_lift_joint
- removed joint shoulder_pan_joint
- removed joint wrist_1_joint
- removed joint wrist_2_joint
- removed joint wrist_3_joint
- removed joint wrist_3_link-tool0_fixed_joint
- added joint left_base_link-base_fixed_joint: type fixed, parent left_base_link, child left_base, origin xyz=0 0 0 rpy=0 0 -3.14159265359
- added joint left_ee_fixed_joint: type fixed, parent left_wrist_3_link, child left_ee_link, origin xyz=0.0 0.0823 0.0 rpy=0.0 0.0 1.57079632679
- added joint left_elbow_joint: type revolute, parent left_upper_arm_link, child left_forearm_link, origin xyz=0.0 -0.1197 0.425 rpy=0.0 0.0 0.0, axis 0 1 0, limit lower=-3.14159265359 upper=3.14159265359 effort=150.0 velocity=3.15
- added joint left_gripper_base_joint: type fixed, parent left_ee_link, child left_gripper_base_link, origin xyz=0 0 0 rpy=0 0 0
- added joint left_gripper_finger1_finger_joint: type fixed, parent left_gripper_finger1_knuckle_link, child left_gripper_finger1_finger_link, origin xyz=-0.00408552455 -0.03148604435 0.0 rpy=0 0 0
- added joint left_gripper_finger1_finger_tip_joint: type continuous, parent left_gripper_finger1_inner_knuckle_link, child left_gripper_finger1_finger_tip_link, origin xyz=0.04303959807 -0.03759940821 0.0 rpy=0.0 0.0 0.0, axis 0 0 1, limit lower=-3.14 upper=3.14 effort=0.1 velocity=100.0, mimic joint=left_gripper_finger1_joint multiplier=-1
- added joint left_gripper_finger1_inner_knuckle_joint: type continuous, parent left_gripper_base_link, child left_gripper_finger1_inner_knuckle_link, origin xyz=0.06142 0.0127 0 rpy=3.14159265359 0.0 0.0, axis 0 0 1, limit lower=-3.14 upper=3.14 effort=0.1 velocity=100.0, mimic joint=left_gripper_finger1_joint offset=0
- added joint left_gripper_finger1_joint: type revolute, parent left_gripper_base_link, child left_gripper_finger1_knuckle_link, origin xyz=0.05490451627 0.03060114443 0.0 rpy=3.14159265359 0.0 0.0, axis 0 0 1, limit lower=0.0 upper=0.804 effort=1000 velocity=2.0
- added joint left_gripper_finger2_finger_joint: type fixed, parent left_gripper_finger2_knuckle_link, child left_gripper_finger2_finger_link, origin xyz=-0.00408552455 -0.03148604435 0.0 rpy=0 0 0
- added joint left_gripper_finger2_finger_tip_joint: type continuous, parent left_gripper_finger2_inner_knuckle_link, child left_gripper_finger2_finger_tip_link, origin xyz=0.04303959807 -0.03759940821  0.0 rpy=0.0 0.0 0.0, axis 0 0 1, limit lower=-3.14 upper=3.14 effort=0.1 velocity=100.0, mimic joint=left_gripper_finger1_joint multiplier=-1
- added joint left_gripper_finger2_inner_knuckle_joint: type continuous, parent left_gripper_base_link, child left_gripper_finger2_inner_knuckle_link, origin xyz=0.06142 -0.0127 0 rpy=0 0 0, axis 0 0 1, limit lower=-3.14 upper=3.14 effort=0.1 velocity=100.0, mimic joint=left_gripper_finger1_joint offset=0
- added joint left_gripper_finger2_joint: type revolute, parent left_gripper_base_link, child left_gripper_finger2_knuckle_link, origin xyz=0.05490451627 -0.03060114443 0.0 rpy=0.0 0.0 0.0, axis 0 0 1, limit lower=-3.14 upper=3.14 effort=1000 velocity=100.0, mimic joint=left_gripper_finger1_joint
- added joint left_shoulder_lift_joint: type revolute, parent left_shoulder_link, child left_upper_arm_link, origin xyz=0.0 0.13585 0.0 rpy=0.0 1.57079632679 0.0, axis 0 1 0, limit lower=-3.14159265359 upper=3.14159265359 effort=150.0 velocity=3.15
- added joint left_shoulder_pan_joint: type revolute, parent left_base_link, child left_shoulder_link, origin xyz=0.0 0.0 0.089159 rpy=0.0 0.0 0.0, axis 0 0 1, limit lower=-3.14159265359 upper=3.14159265359 effort=150.0 velocity=3.15
- added joint left_wrist_1_joint: type revolute, parent left_forearm_link, child left_wrist_1_link, origin xyz=0.0 0.0 0.39225 rpy=0.0 1.57079632679 0.0, axis 0 1 0, limit lower=-3.14159265359 upper=3.14159265359 effort=28.0 velocity=3.2
- added joint left_wrist_2_joint: type revolute, parent left_wrist_1_link, child left_wrist_2_link, origin xyz=0.0 0.093 0.0 rpy=0.0 0.0 0.0, axis 0 0 1, limit lower=-3.14159265359 upper=3.14159265359 effort=28.0 velocity=3.2
- added joint left_wrist_3_joint: type revolute, parent left_wrist_2_link, child left_wrist_3_link, origin xyz=0.0 0.0 0.09465 rpy=0.0 0.0 0.0, axis 0 1 0, limit lower=-3.14159265359 upper=3.14159265359 effort=28.0 velocity=3.2
- added joint left_wrist_3_link-tool0_fixed_joint: type fixed, parent left_wrist_3_link, child left_tool0, origin xyz=0 0.0823 0 rpy=-1.57079632679 0 0
- added joint right_base_link-base_fixed_joint: type fixed, parent right_base_link, child right_base, origin xyz=0 0 0 rpy=0 0 -3.14159265359
- added joint right_ee_fixed_joint: type fixed, parent right_wrist_3_link, child right_ee_link, origin xyz=0.0 0.0823 0.0 rpy=0.0 0.0 1.57079632679
- added joint right_elbow_joint: type revolute, parent right_upper_arm_link, child right_forearm_link, origin xyz=0.0 -0.1197 0.425 rpy=0.0 0.0 0.0, axis 0 1 0, limit lower=-3.14159265359 upper=3.14159265359 effort=150.0 velocity=3.15
- added joint right_gripper_base_joint: type fixed, parent right_ee_link, child right_gripper_base_link, origin xyz=0 0 0 rpy=0 0 0
- added joint right_gripper_finger1_finger_joint: type fixed, parent right_gripper_finger1_knuckle_link, child right_gripper_finger1_finger_link, origin xyz=-0.00408552455 -0.03148604435 0.0 rpy=0 0 0
- added joint right_gripper_finger1_finger_tip_joint: type continuous, parent right_gripper_finger1_inner_knuckle_link, child right_gripper_finger1_finger_tip_link, origin xyz=0.04303959807 -0.03759940821 0.0 rpy=0.0 0.0 0.0, axis 0 0 1, limit lower=-3.14 upper=3.14 effort=0.1 velocity=100.0, mimic joint=right_gripper_finger1_joint multiplier=-1
- added joint right_gripper_finger1_inner_knuckle_joint: type continuous, parent right_gripper_base_link, child right_gripper_finger1_inner_knuckle_link, origin xyz=0.06142 0.0127 0 rpy=3.14159265359 0.0 0.0, axis 0 0 1, limit lower=-3.14 upper=3.14 effort=0.1 velocity=100.0, mimic joint=right_gripper_finger1_joint offset=0
- added joint right_gripper_finger1_joint: type revolute, parent right_gripper_base_link, child right_gripper_finger1_knuckle_link, origin xyz=0.05490451627 0.03060114443 0.0 rpy=3.14159265359 0.0 0.0, axis 0 0 1, limit lower=0.0 upper=0.804 effort=1000 velocity=2.0
- added joint right_gripper_finger2_finger_joint: type fixed, parent right_gripper_finger2_knuckle_link, child right_gripper_finger2_finger_link, origin xyz=-0.00408552455 -0.03148604435 0.0 rpy=0 0 0
- added joint right_gripper_finger2_finger_tip_joint: type continuous, parent right_gripper_finger2_inner_knuckle_link, child right_gripper_finger2_finger_tip_link, origin xyz=0.04303959807 -0.03759940821  0.0 rpy=0.0 0.0 0.0, axis 0 0 1, limit lower=-3.14 upper=3.14 effort=0.1 velocity=100.0, mimic joint=right_gripper_finger1_joint multiplier=-1
- added joint right_gripper_finger2_inner_knuckle_joint: type continuous, parent right_gripper_base_link, child right_gripper_finger2_inner_knuckle_link, origin xyz=0.06142 -0.0127 0 rpy=0 0 0, axis 0 0 1, limit lower=-3.14 upper=3.14 effort=0.1 velocity=100.0, mimic joint=right_gripper_finger1_joint offset=0
- added joint right_gripper_finger2_joint: type revolute, parent right_gripper_base_link, child right_gripper_finger2_knuckle_link, origin xyz=0.05490451627 -0.03060114443 0.0 rpy=0.0 0.0 0.0, axis 0 0 1, limit lower=-3.14 upper=3.14 effort=1000 velocity=100.0, mimic joint=right_gripper_finger1_joint
- added joint right_shoulder_lift_joint: type revolute, parent right_shoulder_link, child right_upper_arm_link, origin xyz=0.0 0.13585 0.0 rpy=0.0 1.57079632679 0.0, axis 0 1 0, limit lower=-3.14159265359 upper=3.14159265359 effort=150.0 velocity=3.15
- added joint right_shoulder_pan_joint: type revolute, parent right_base_link, child right_shoulder_link, origin xyz=0.0 0.0 0.089159 rpy=0.0 0.0 0.0, axis 0 0 1, limit lower=-3.14159265359 upper=3.14159265359 effort=150.0 velocity=3.15
- added joint right_wrist_1_joint: type revolute, parent right_forearm_link, child right_wrist_1_link, origin xyz=0.0 0.0 0.39225 rpy=0.0 1.57079632679 0.0, axis 0 1 0, limit lower=-3.14159265359 upper=3.14159265359 effort=28.0 velocity=3.2
- added joint right_wrist_2_joint: type revolute, parent right_wrist_1_link, child right_wrist_2_link, origin xyz=0.0 0.093 0.0 rpy=0.0 0.0 0.0, axis 0 0 1, limit lower=-3.14159265359 upper=3.14159265359 effort=28.0 velocity=3.2
- added joint right_wrist_3_joint: type revolute, parent right_wrist_2_link, child right_wrist_3_link, origin xyz=0.0 0.0 0.09465 rpy=0.0 0.0 0.0, axis 0 1 0, limit lower=-3.14159265359 upper=3.14159265359 effort=28.0 velocity=3.2
- added joint right_wrist_3_link-tool0_fixed_joint: type fixed, parent right_wrist_3_link, child right_tool0, origin xyz=0 0.0823 0 rpy=-1.57079632679 0 0
- joint world_joint_1: child base_link -> left_base_link
- joint world_joint_2: child 2_base_link -> right_base_link

Commit message: able to show ur5Frame in gazebo

File: ur5_dual_arm_tufts/urdf/ur5_dual_arm.xacro (robot description, xacro)
@@ -28,6 +28,6 @@
   <link name="ur5_frame">
     <inertial>
-      <origin rpy  ="0.0 0 0" xyz="0 0 0"/>
-      <mass value="27.2155"/>
+      <origin rpy  ="0.0 0 0" xyz="0.0 0.0 0.0"/>
+      <mass value="27.21"/>
       <inertia
         ixx="5.01" ixy="0.0" ixz="0.0"
@@ -44,5 +44,6 @@
       <origin rpy="0.0 0 0" xyz="0 0 0"/>
       <geometry>
-        <mesh filename="package://ur5_dual_arm_tufts/meshes/UR5Frame.dae"/>
+        <mesh filename="package://ur5_dual_arm_tufts/meshes/UR5Frame.STL"/>
+        <!-- <mesh filename="/home/andrecleaver/catkin_ws/src/Hacking-SotA-UR5/ur5_dual_arm_tufts/meshes/UR5Frame.dae"/> -->
       </geometry>
     </visual>

Commit message: add collision to urdf dual arm

File: ur5_dual_arm_tufts/urdf/ur5_dual_arm.xacro (robot description, xacro)
@@ -35,10 +35,10 @@
         izz="3.20"/>
     </inertial>
-<!--     <collision>
+    <collision>
       <origin rpy="0.0 0 0" xyz="0 0 0"/>
       <geometry>
-        <mesh filename="package://ur5_dual_arm_tufts/meshes/UR5Frame.dae"/>
+        <mesh filename="package://ur5_dual_arm_tufts/meshes/UR5Frame.stl"/>
       </geometry>
-    </collision> -->
+    </collision>
     <visual>
       <origin rpy="0.0 0 0" xyz="0 0 0"/>
